File: pcb/rp2040_devboard.kicad_sch (KiCad schematic)
At the start: 33 parts, among them J1 USB_C_Receptacle_USB2.0_14P, J2 Conn_01x20, J3 Conn_01x20, J4 Conn_01x03, SW1 SW_Push, U1 RP2040, U3 W25Q128JVS, U4 MCP1700x-330xxTT, Y1 12MHz

Commit message: added readme, working on journals
Parts:
- added U2: OLED_0.49_SSD1306_I2C, Display:ER_OLEDM0.91_1x-I2C, symbol Display_Graphic:ER_OLEDM0.91_1x-I2C
Connections:
- net +3V3: now also U2.2 (VCC)
- net GND: now also U2.1 (GND)
- net GPIO0: now also U2.3 (SCL)
- net GPIO1: now also U2.4 (SDA)
Other:
- note added: "RP2040 devboard with OLED"
- note removed: "Custom RP2040 devboard"
- moved on the sheet: C1, C10, C11, C12, C15, C16, C17, C2, C3, C4, C5, C6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
